File: noritake_mn12864k_vfd_breakout.kicad_pcb (KiCad board)
At the start: 4 copper layers, 100 x 56 mm, 30 parts, among them J1 Conn_01x14, T1 Wuerth 760390013, U1 XL6007E1, U2 SN6501, U3 SN74AVC8T245PW, U4 MN12864K, U5 SN74AVC8T245PW

Commit message: Finish layout for assembly
Parts:
- added H1: MountingHole, ToolingHole:ToolingHole_JLCSMT, F.Cu at (199.0, 155.0)
- added H2: MountingHole, ToolingHole:ToolingHole_JLCSMT, F.Cu at (101.0, 101.0)
Routing:
- net /F1: track 92.6 -> 91.9 mm, vias 4 -> 3
- net GND: vias 22 -> 124
- net +5V: vias 22 -> 24
Other:
- board text added: "JLCJLCJLCJLC"
- board text added: "Noritake MN12864K VFD Breadboard adapter Rev A 2020 Designed by Tobias Schramm"
- board text removed: "VFD Breadboard adapter Noritake MN12864K RevA"
