File: noritake_mn12864k_vfd_breakout.sch (KiCad schematic (older format))
At the start: 30 parts, among them J1 Conn_01x14, T1 Wuerth 760390013, U1 XL6007E1, U2 SN6501, U3 SN74AVC8T245PW, U4 MN12864K, U5 SN74AVC8T245PW

Commit message: Finish layout for assembly
Parts:
- added H1, H2: MountingHole, ToolingHole:ToolingHole_JLCSMT, symbol Mechanical:MountingHole
- U2: Field4 (none) -> C49451
- U3, U5: LCSC (none) -> C7859
Changed lines of the file:
@@
 F 2 "Package_SO:TSSOP-24_4.4x7.8mm_P0.65mm" H 7850 1450 50  0001 C CNN
 F 3 "https://www.ti.com/lit/ds/symlink/sn74avc8t245.pdf" H 6900 1850 50  0001 C CNN
+F 4 "C7859" V 6950 2100 50  0001 C CNN "LCSC"
 	1    6950 2100
 	-1   0    0    -1
@@
 F 2 "Package_SO:TSSOP-24_4.4x7.8mm_P0.65mm" H 10800 1450 50  0001 C CNN
 F 3 "https://www.ti.com/lit/ds/symlink/sn74avc8t245.pdf" H 9850 1850 50  0001 C CNN
+F 4 "C7859" V 9900 2100 50  0001 C CNN "LCSC"
 	1    9900 2100
 	1    0    0    -1
@@
 F 2 "Package_TO_SOT_SMD:SOT-23-5" H 2800 7050 50  0001 C CNN
 F 3 "http://www.ti.com/lit/ds/symlink/sn6501.pdf" H 2800 7050 50  0001 C CNN
+F 4 "C49451" H 2800 6700 50  0001 C CNN "Field4"
 	1    2800 6700
 	1    0    0    -1
@@
 Wire Wire Line
 	6400 1300 6500 1300
+$Comp
+L Mechanical:MountingHole H2
+U 1 1 5F61E373
+P 10550 6350
+F 0 "H2" H 10650 6396 50  0000 L CNN
+F 1 "MountingHole" H 10650 6305 50  0000 L CNN
+F 2 "ToolingHole:ToolingHole_JLCSMT" H 10550 6350 50  0001 C CNN
+F 3 "~" H 10550 6350 50  0001 C CNN
+	1    10550 6350
+	1    0    0    -1
+$EndComp
+$Comp
+L Mechanical:MountingHole H1
+U 1 1 5F61F352
+P 10550 6150
+F 0 "H1" H 10650 6196 50  0000 L CNN
+F 1 "MountingHole" H 10650 6105 50  0000 L CNN
+F 2 "ToolingHole:ToolingHole_JLCSMT" H 10550 6150 50  0001 C CNN
+F 3 "~" H 10550 6150 50  0001 C CNN
+	1    10550 6150
+	1    0    0    -1
+$EndComp
 $EndSCHEMATC

Commit message: Fix 1kR LCSC partnumber
Parts:
- R5: LCSC C25905 -> C11702
Changed lines of the file:
@@
 F 2 "Resistor_SMD:R_0402_1005Metric" V 4480 2850 50  0001 C CNN
 F 3 "https://datasheet.lcsc.com/szlcsc/Uniroyal-Elec-0402WGF5101TCE_C25905.pdf" H 4550 2850 50  0001 C CNN
-F 4 "C25905" H 4550 2850 50  0001 C CNN "LCSC"
+F 4 "C11702" H 4550 2850 50  0001 C CNN "LCSC"
 	1    4550 2850
 	1    0    0    -1
